File: EF_matrix.kicad_sch (KiCad schematic)
At the start: 16 parts, among them J2 Conn_02x05_Counter_Clockwise, J21 Conn_01x01_Socket, J27 Conn_01x01_Socket, J28 Conn_01x01_Socket

Commit message: Minor optical fixes
Other:
- note added: "LED Panel"
- note removed: "Button & LED Panel"
- moved on the sheet: J27, J28
