File: xlr_input.kicad_sch (KiCad schematic)
At the start: 6 parts, among them J1 XLR3, J2 XLR3, J21 Conn_01x01_Socket, J3 XLR3, J4 XLR3

Commit message: Finished up PCB layout
Parts:
- removed J1, J2, J3, J4: XLR3, symbol Connector_Audio:XLR3
- added J11, J5, J7, J9: NC3FAAV2, Connector_Audio:Jack_XLR_Neutrik_NC3FAAV2_Vertical, symbol Connector_Audio:NC3FAAV2
Connections:
- net Channel 1 Cold: now also J5.3
- net Channel 1 Hot: now also J5.2
- net Channel 2 Cold: now also J7.3
- net Channel 2 Hot: now also J7.2
- net Channel 3 Cold: now also J9.3
- net Channel 3 Hot: now also J9.2
- net Channel 4 Cold: now also J11.3
- net Channel 4 Hot: now also J11.2
- net Pin1: now reaches J21.1 (Pin_1)
- net Pin1: now also J11.1, J5.1, J7.1, J9.1
- no-connect marks 0 -> 4
