File: xlr_output.kicad_sch (KiCad schematic)
At the start: 6 parts, among them J1 XLR3, J2 XLR3, J21 Conn_01x01_Socket, J3 XLR3, J4 XLR3

Commit message: Finished up PCB layout
Parts:
- removed J1, J2, J3, J4: XLR3, symbol Connector_Audio:XLR3
- added J13, J14, J15, J16: NC3MAAH, Connector_Audio:Jack_XLR_Neutrik_NC3MAAV_Vertical, symbol Connector_Audio:NC3MAAV
Connections:
- net Channel 1 Cold: now also J13.3
- net Channel 1 Hot: now also J13.2
- net Channel 2 Cold: now also J14.3
- net Channel 2 Hot: now also J14.2
- net Channel 3 Cold: now also J15.3
- net Channel 3 Hot: now also J15.2
- net Channel 4 Cold: now also J16.3
- net Channel 4 Hot: now also J16.2
- net Pin1: now reaches J21.1 (Pin_1)
- net Pin1: now also J13.1, J14.1, J15.1, J16.1
- no-connect marks 0 -> 4
