File: EF_matrix.kicad_pcb (KiCad board)
At the start: 2 copper layers, 170.2 x 149.9 mm, 80 parts, among them J1 Conn_02x05_Counter_Clockwise, J10 NC3FAAV2, J11 NC3FAAV2, J12 NC3FAAV2, J13 NC3MAAH, J14 NC3MAAH, J15 NC3MAAH, J16 NC3MAAH, J17 Conn_02x05_Counter_Clockwise, J18 Conn_02x05_Counter_Clockwise, J19 Conn_02x05_Counter_Clockwise, J2 Conn_01x01_Socket, J20 Conn_02x05_Counter_Clockwise, J22 Conn_01x01_Socket, J23 Conn_01x01_Socket, J25 Conn_01x01_Socket, J26 Conn_01x01_Socket, J3 Conn_02x05_Counter_Clockwise, J31 Conn_02x05_Counter_Clockwise, J32 Conn_01x01_Socket, J33 Conn_01x01_Socket, J34 Conn_01x01_Socket, J35 Conn_01x01_Socket, J36 Conn_01x01_Socket, J37 Conn_01x01_Socket, J38 Conn_01x01_Socket, J39 Conn_01x01_Socket, J4 Conn_02x05_Counter_Clockwise, J40 Conn_01x01_Socket, J5 NC3FAAV2, J6 NC3FAAV2, J7 NC3FAAV2, J8 NC3FAAV2, J9 NC3FAAV2, K1 G5V-2, K2 G5V-2, K3 G5V-2, K4 G5V-2, K5 G5V-2, K6 G5V-2, K7 G5V-2, K8 G5V-2

Commit message: splitting out single pcb files for production
Parts:
- moved JP5 156.6 mm to (277.7, 81.8), turned to -90 degrees
- moved JP1 153.3 mm to (277.7, 89.1), turned to -90 degrees
- moved D5 152.7 mm to (272.6, 76.4), turned to 180 degrees
- moved REF** 141.2 mm to (273.6, 124.1), turned to 0 degrees
- moved K1 140.3 mm to (265.0, 81.0), turned to 0 degrees
- moved REF** 134.3 mm to (257.1, 74.6), turned to 0 degrees
- moved JP13 133.4 mm to (259.9, 81.5), turned to 90 degrees
- moved JP9 129.3 mm to (259.9, 89.4), turned to -90 degrees
- moved J19 128.4 mm to (264.0, 109.7), turned to 90 degrees
- moved JP6 126.4 mm to (254.5, 81.8), turned to -90 degrees
- moved D6 123.6 mm to (249.5, 76.4), turned to 180 degrees
- moved JP2 122.2 mm to (254.5, 89.3), turned to -90 degrees
- moved K3 111.0 mm to (241.8, 81.0), turned to 0 degrees
- moved JP14 104.3 mm to (236.8, 81.8), turned to 90 degrees
- moved JP10 99.2 mm to (236.8, 89.3), turned to -90 degrees
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Other:
- board size 170.2 x 149.9 mm -> 268.6 x 182.9 mm
- board text added: "+"
- board text added: "-"
- board text added: "GND Lift"
- board text added: "In 1"
- board text added: "In 2"
- board text added: "Mute"
- board text added: "Mute GND"
- board text added: "Mute H/C"
- board text added: "Power"
